File: board-1.sch (KiCad schematic (older format))
At the start: 19 parts, among them P1 RESET, P2 USB, P3 CONN_01X07, P4 CONN_01X05, P5 CONN_01X02, U1 MCP1700, U2 PIC32MX2XX, Y1 24MHz

Commit message: Added diode between USB power in and voltage regulator.
Also added OSHW logo.
Parts:
- added C7: 47uF, Capacitors_ThroughHole:C_Radial_D5_L6_P2.5, symbol CP
- added D2: D, Diodes_ThroughHole:Diode_DO-35_SOD27_Horizontal_RM10, symbol D
Connections:
- net +3V3: now also C7.1
- net GND: now also C7.2
- net UART_RCV: now also P5.1 (P1), U2.3 (RA1); no longer P5.2 (P2), U2.4 (RB0)
- net UART_SND: now also P5.2 (P2), U2.4 (RB0); no longer P5.1 (P1), U2.3 (RA1)
- net at U1.2 (VIN), U2.15 (VBUS): now also D2.1 (K); no longer P2.1 (VCC)
- net at U2.24 (RB13): now also P4.2 (P2); no longer P4.5 (P5)
- net at U2.25 (RB14): now also P4.5 (P5); no longer P4.1 (P1)
- net at U2.26 (RB15): now also P4.1 (P1); no longer P4.2 (P2)
- new net: D2.2 (A), P2.1 (VCC)
Changed lines of the file:
@@
 L +3V3 #PWR07
 U 1 1 5688E4AA
-P 4800 3850
-F 0 "#PWR07" H 4800 3700 50  0001 C CNN
-F 1 "+3V3" H 4650 3900 50  0000 C CNN
-F 2 "" H 4800 3850 50  0000 C CNN
-F 3 "" H 4800 3850 50  0000 C CNN
-	1    4800 3850
-	0    -1   -1   0
+P 4500 3850
+F 0 "#PWR07" H 4500 3700 50  0001 C CNN
+F 1 "+3V3" H 4350 3900 50  0000 C CNN
+F 2 "" H 4500 3850 50  0000 C CNN
+F 3 "" H 4500 3850 50  0000 C CNN
+	1    4500 3850
+	1    0    0    -1
 $EndComp
 $Comp
@@
 	3500 3300 4100 3300
 Wire Wire Line
-	3500 3600 3900 3600
-Wire Wire Line
-	3500 3500 4000 3500
-Wire Wire Line
 	1400 3000 1800 3000
 Wire Wire Line
@@
 	1900 3500 1900 3350
 Connection ~ 1700 3350
-Connection ~ 1200 2250
-Wire Wire Line
-	1200 1550 1200 2600
 Wire Wire Line
 	1700 2500 1700 2700
@@
 	1    0    0    -1
 $EndComp
-Wire Wire Line
-	4700 3300 4900 3300
 $Comp
 L +3V3 #PWR013
@@
 	3850 2300 3850 2150
 Text Label 3550 2300 0    60   ~ 0
-UART_RCV
+UART_SND
 Wire Wire Line
 	3850 2050 3500 2050
 Text Label 3500 2050 0    60   ~ 0
-UART_SND
+UART_RCV
 Wire Wire Line
 	2000 3400 1950 3400
@@
 	1950 3800 1700 3800
 Text Label 1700 3800 0    60   ~ 0
-UART_SND
+UART_RCV
 $Comp
 L CONN_01X05 P4
@@
 $EndComp
 Wire Wire Line
-	3500 3400 3500 3950
-Wire Wire Line
-	3500 3950 4900 3950
-Wire Wire Line
-	4800 3850 4900 3850
-Wire Wire Line
-	4700 3300 4700 3750
-Connection ~ 4850 3300
-Wire Wire Line
-	4700 3750 4900 3750
-Wire Wire Line
-	4900 3550 4000 3550
-Wire Wire Line
-	4000 3550 4000 3500
-Wire Wire Line
-	4900 3650 3900 3650
-Wire Wire Line
-	3900 3650 3900 3600
+	4500 3850 4900 3850
 Wire Wire Line
 	1250 3950 1250 4300
@@
 	1050 4650 1250 4650
 Connection ~ 1250 4650
+Wire Wire Line
+	3700 3950 4900 3950
+Wire Wire Line
+	3700 3500 3700 3950
+Wire Wire Line
+	3700 3500 3500 3500
+Wire Wire Line
+	4900 3650 4000 3650
+Wire Wire Line
+	4000 3650 4000 3400
+Wire Wire Line
+	4000 3400 3500 3400
+Wire Wire Line
+	4900 3550 3600 3550
+Wire Wire Line
+	3600 3550 3600 3600
+Wire Wire Line
+	3600 3600 3500 3600
+Wire Wire Line
+	4850 3300 4900 3300
+Wire Wire Line
+	4900 3750 4750 3750
+Wire Wire Line
+	4750 3750 4750 4050
+$Comp
+L GND #PWR014
+U 1 1 56AD61B0
+P 4750 4050
+F 0 "#PWR014" H 4750 3800 50  0001 C CNN
+F 1 "GND" H 4758 3876 50  0000 C CNN
+F 2 "" H 4750 4050 50  0000 C CNN
+F 3 "" H 4750 4050 50  0000 C CNN
+	1    4750 4050
+	1    0    0    -1
+$EndComp
+$Comp
+L CP C7
+U 1 1 56AD66F2
+P 1250 950
+F 0 "C7" H 1368 996 50  0000 L CNN
+F 1 "47uF" H 1368 904 50  0000 L CNN
+F 2 "Capacitors_ThroughHole:C_Radial_D5_L6_P2.5" H 1288 800 50  0001 C CNN
+F 3 "" H 1250 950 50  0000 C CNN
+	1    1250 950
+	1    0    0    -1
+$EndComp
+$Comp
+L GND #PWR015
+U 1 1 56AD6750
+P 1250 1200
+F 0 "#PWR015" H 1250 950 50  0001 C CNN
+F 1 "GND" H 1258 1026 50  0000 C CNN
+F 2 "" H 1250 1200 50  0000 C CNN
+F 3 "" H 1250 1200 50  0000 C CNN
+	1    1250 1200
+	1    0    0    -1
+$EndComp
+Wire Wire Line
+	1250 1100 1250 1200
+Wire Wire Line
+	1000 800  1250 800
+Connection ~ 1000 800
+$Comp
+L D D2
+U 1 1 56B145BA
+P 1200 1900
+F 0 "D2" V 1246 1822 50  0000 R CNN
+F 1 "D" V 1154 1822 50  0000 R CNN
+F 2 "Diodes_ThroughHole:Diode_DO-35_SOD27_Horizontal_RM10" H 1200 1900 50  0001 C CNN
+F 3 "" H 1200 1900 50  0000 C CNN
+	1    1200 1900
+	0    -1   -1   0
+$EndComp
+Wire Wire Line
+	1200 2050 1200 2600
+Wire Wire Line
+	1200 1750 1200 1550
+Connection ~ 1200 2250
 $EndSCHEMATC

Commit message: Revision 3.
Parts:
- removed P1: RESET, Pin_Headers:Pin_Header_Straight_1x02, symbol CONN_01X02
- removed P2: USB, footprint:USB_B, symbol USB_B
- added P1: CONN_01X03, Pin_Headers:Pin_Header_Straight_1x03, symbol CONN_01X03
- added P2: USB_B_fixed, footprint:USB_B, symbol USB_B_fixed
- R1, R2, R4: footprint Resistors_ThroughHole:Resistor_Horizontal_RM15mm -> Resistors_ThroughHole:Resistor_Horizontal_RM10mm
Connections:
- net labels added: USB_N, USB_P
- net labels removed: USB_DN, USB_DP
- wire segments 88 -> 87
- no-connect marks 6 -> 4
Changed lines of the file:
@@
 $EndDescr
-$Comp
-L USB_B P2
-U 1 1 5688ADEE
-P 1650 1250
-F 0 "P2" H 1673 1582 50  0000 C CNN
-F 1 "USB" H 1673 1490 50  0000 C CNN
-F 2 "footprint:USB_B" V 1600 1150 50  0000 C CNN
-F 3 "" V 1600 1150 50  0000 C CNN
-	1    1650 1250
-	1    0    0    -1
-$EndComp
-$Comp
-L CONN_01X02 P1
-U 1 1 5688AE71
-P 850 4450
-F 0 "P1" H 927 4488 50  0000 L CNN
-F 1 "RESET" H 927 4396 50  0000 L CNN
-F 2 "Pin_Headers:Pin_Header_Straight_1x02" H 850 4450 50  0001 C CNN
-F 3 "" H 850 4450 50  0000 C CNN
-	1    850  4450
-	-1   0    0    1
-$EndComp
 $Comp
 L PIC32MX2XX U2
@@
 F 0 "R2" V 1292 3950 50  0000 C CNN
 F 1 "470" V 1384 3950 50  0000 C CNN
-F 2 "Resistors_ThroughHole:Resistor_Horizontal_RM15mm" V 1430 3950 50  0000 C CNN
+F 2 "Resistors_ThroughHole:Resistor_Horizontal_RM10mm" V 1430 3950 50  0000 C CNN
 F 3 "" H 1500 3950 50  0000 C CNN
 	1    1500 3950
@@
 F 0 "R1" V 1208 3950 50  0000 C CNN
 F 1 "10K" V 1116 3950 50  0000 C CNN
-F 2 "Resistors_ThroughHole:Resistor_Horizontal_RM15mm" V 930 3950 50  0000 C CNN
+F 2 "Resistors_ThroughHole:Resistor_Horizontal_RM10mm" V 930 3950 50  0000 C CNN
 F 3 "" H 1000 3950 50  0000 C CNN
 	1    1000 3950
@@
 $EndComp
 Text Label 2100 1750 0    60   ~ 0
-USB_DN
+USB_N
 Text Label 2100 1650 0    60   ~ 0
-USB_DP
+USB_P
 Text Label 4100 3200 0    60   ~ 0
-USB_DP
+USB_P
 Text Label 4100 3300 0    60   ~ 0
-USB_DN
+USB_N
 $Comp
 L +3V3 #PWR07
@@
 NoConn ~ 3500 2700
 NoConn ~ 3500 2600
-NoConn ~ 3500 2500
-NoConn ~ 3500 2400
 NoConn ~ 2000 3700
 $Comp
@@
 F 0 "R4" V 2492 4500 50  0000 C CNN
 F 1 "330" V 2584 4500 50  0000 C CNN
-F 2 "Resistors_ThroughHole:Resistor_Horizontal_RM15mm" V 2630 4500 50  0001 C CNN
+F 2 "Resistors_ThroughHole:Resistor_Horizontal_RM10mm" V 2630 4500 50  0001 C CNN
 F 3 "" H 2700 4500 50  0000 C CNN
 	1    2700 4500
@@
 $EndComp
 Wire Wire Line
-	4900 2700 4850 2700
+	4000 2700 4900 2700
 Wire Wire Line
 	4850 2700 4850 2350
@@
 	1250 3950 1250 4300
 Wire Wire Line
-	1050 4250 1050 4400
-Wire Wire Line
-	1050 4250 1250 4250
-Connection ~ 1250 4250
-Wire Wire Line
-	1050 4500 1050 4650
-Wire Wire Line
-	1050 4650 1250 4650
-Connection ~ 1250 4650
-Wire Wire Line
 	3700 3950 4900 3950
 Wire Wire Line
@@
 	1200 1750 1200 1550
 Connection ~ 1200 2250
+$Comp
+L USB_B_fixed P2
+U 1 1 56CA5BB4
+P 1650 1250
+F 0 "P2" H 1673 1582 50  0000 C CNN
+F 1 "USB_B_fixed" H 1673 1490 50  0000 C CNN
+F 2 "footprint:USB_B" V 1600 1150 50  0001 C CNN
+F 3 "" V 1600 1150 50  0000 C CNN
+	1    1650 1250
+	1    0    0    -1
+$EndComp
+$Comp
+L CONN_01X03 P1
+U 1 1 57416384
+P 4200 2500
+F 0 "P1" H 4277 2538 50  0000 L CNN
+F 1 "CONN_01X03" H 4277 2446 50  0000 L CNN
+F 2 "Pin_Headers:Pin_Header_Straight_1x03" H 4200 2500 50  0001 C CNN
+F 3 "" H 4200 2500 50  0000 C CNN
+	1    4200 2500
+	1    0    0    -1
+$EndComp
+Wire Wire Line
+	3500 2400 4000 2400
+Wire Wire Line
+	3500 2500 4000 2500
+Wire Wire Line
+	4000 2600 4000 2700
+Connection ~ 4850 2700
 $EndSCHEMATC

Commit message: Updated capacitor footprints.
Parts:
- C1, C2, C3, C4, C5, C6: footprint Capacitors_ThroughHole:C_Disc_D6_P5 -> Capacitors_ThroughHole:C_Rect_L7_W2.5_P5
- U1: footprint Housings_TO-92:TO-92_Inline_Narrow_Oval -> Housings_TO-92:TO-92_Inline_Wide
Changed lines of the file:
@@
 F 0 "C1" V 797 3150 50  0000 C CNN
 F 1 "10uF (low ESR)" V 889 3150 50  0000 C CNN
-F 2 "Capacitors_ThroughHole:C_Disc_D6_P5" H 1088 3000 50  0001 C CNN
+F 2 "Capacitors_ThroughHole:C_Rect_L7_W2.5_P5" H 1088 3000 50  0001 C CNN
 F 3 "" H 1050 3150 50  0000 C CNN
 F 4 "Low-ESR" V 1050 3150 60  0001 C CNN "Notes"
@@
 F 0 "C2" H 1365 4496 50  0000 L CNN
 F 1 "100nF" H 1365 4404 50  0000 L CNN
-F 2 "Capacitors_ThroughHole:C_Disc_D6_P5" H 1288 4300 50  0001 C CNN
+F 2 "Capacitors_ThroughHole:C_Rect_L7_W2.5_P5" H 1288 4300 50  0001 C CNN
 F 3 "" H 1250 4450 50  0000 C CNN
 	1    1250 4450
@@
 F 0 "C3" H 1400 3000 50  0000 L CNN
 F 1 "100nF (low ESR)" H 1250 2950 50  0000 L CNN
-F 2 "Capacitors_ThroughHole:C_Disc_D6_P5" H 1438 2700 50  0001 C CNN
+F 2 "Capacitors_ThroughHole:C_Rect_L7_W2.5_P5" H 1438 2700 50  0001 C CNN
 F 3 "" H 1400 2850 50  0000 C CNN
 	1    1400 2850
@@
 F 0 "C4" H 1815 2896 50  0000 L CNN
 F 1 "100nF (low ESR)" H 1550 3050 50  0000 L CNN
-F 2 "Capacitors_ThroughHole:C_Disc_D6_P5" H 1738 2700 50  0001 C CNN
+F 2 "Capacitors_ThroughHole:C_Rect_L7_W2.5_P5" H 1738 2700 50  0001 C CNN
 F 3 "" H 1700 2850 50  0000 C CNN
 	1    1700 2850
@@
 F 0 "U1" V 1006 1272 60  0000 R CNN
 F 1 "MCP1700" V 900 1272 60  0000 R CNN
-F 2 "Housings_TO-92:TO-92_Inline_Narrow_Oval" V 794 1272 60  0000 R CNN
+F 2 "Housings_TO-92:TO-92_Inline_Wide" V 794 1272 60  0000 R CNN
 F 3 "" H 900 1500 60  0000 C CNN
 	1    900  1500
@@
 F 0 "C5" V 1100 3400 50  0000 C CNN
 F 1 "33pF" V 1200 3400 50  0000 C CNN
-F 2 "Capacitors_ThroughHole:C_Disc_D6_P5" H 1388 3250 50  0001 C CNN
+F 2 "Capacitors_ThroughHole:C_Rect_L7_W2.5_P5" H 1388 3250 50  0001 C CNN
 F 3 "" H 1350 3400 50  0000 C CNN
 	1    1350 3400
@@
 F 0 "C6" V 1300 3600 50  0000 C CNN
 F 1 "33pF" V 1400 3600 50  0000 C CNN
-F 2 "Capacitors_ThroughHole:C_Disc_D6_P5" H 1388 3450 50  0001 C CNN
+F 2 "Capacitors_ThroughHole:C_Rect_L7_W2.5_P5" H 1388 3450 50  0001 C CNN
 F 3 "" H 1350 3600 50  0000 C CNN
 	1    1350 3600
